Commit message: fix

File: src/ackermann_nav/urdf/ackermann.urdf.xacro (robot description, xacro)
@@ -2,9 +2,9 @@
 <robot name="ackermann_robot" xmlns:xacro="http://www.ros.org/wiki/xacro">
   <!-- 机器人参数 -->
-  <xacro:property name="base_length" value="0.5"/>
-  <xacro:property name="base_width" value="0.3"/>
-  <xacro:property name="base_height" value="0.1"/>
-  <xacro:property name="wheel_radius" value="0.1"/>
-  <xacro:property name="wheel_width" value="0.05"/>
+  <xacro:property name="base_length" value="0.35"/>
+  <xacro:property name="base_width" value="0.19"/>
+  <xacro:property name="base_height" value="0.20"/>
+  <xacro:property name="wheel_radius" value="0.035"/>
+  <xacro:property name="wheel_width" value="0.03"/>
   <!-- 底盘link -->
   <link name="base_link">
